Commit message: Chage dir name

File: myrobot_sim_gazebo/urdf/LeKiwi3.urdf (robot description, URDF)
Before this commit: robot LeKiwi, 46 links, 45 joints
Links:
- link 4-Omni-Directional-Wheel_Single_Body-v1: geometry collision mesh filename=package://myrobot_sim_gazebo/urdf/meshes/4-Omni-Directional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 scale=0.001 0.001 0.001; visual mesh filename=package://myrobot_sim_gazebo/urdf/meshes/4-Omni-Directional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 scale=0.001 0.001 0.001
- link 4-Omni-Directional-Wheel_Single_Body-v1-1: geometry collision mesh filename=package://myrobot_sim_gazebo/urdf/meshes/4-Omni-Directional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 scale=0.001 0.001 0.001; visual mesh filename=package://myrobot_sim_gazebo/urdf/meshes/4-Omni-Directional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 scale=0.001 0.001 0.001
- link 4-Omni-Directional-Wheel_Single_Body-v1-2: geometry collision mesh filename=package://myrobot_sim_gazebo/urdf/meshes/4-Omni-Directional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 scale=0.001 0.001 0.001; visual mesh filename=package://myrobot_sim_gazebo/urdf/meshes/4-Omni-Directional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 scale=0.001 0.001 0.001
- link 94868A713_NO-THREADS_Female-Threaded-Hex-Standoff: geometry collision mesh filename=package://myrobot_sim_gazebo/urdf/meshes/94868A713_NO-THREA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 scale=0.001 0.001 0.001; visual mesh filename=package://myrobot_sim_gazebo/urdf/meshes/94868A713_NO-THREA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 scale=0.001 0.001 0.001
- link 94868A713_NO-THREADS_Female-Threaded-Hex-Standoff-1: geometry collision mesh filename=package://myrobot_sim_gazebo/urdf/meshes/94868A713_NO-THREA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 scale=0.001 0.001 0.001; visual mesh filename=package://myrobot_sim_gazebo/urdf/meshes/94868A713_NO-THREA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 scale=0.001 0.001 0.001
- link 94868A713_NO-THREADS_Female-Threaded-Hex-Standoff-2: geometry collision mesh filename=package://myrobot_sim_gazebo/urdf/meshes/94868A713_NO-THREA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 scale=0.001 0.001 0.001; visual mesh filename=package://myrobot_sim_gazebo/urdf/meshes/94868A713_NO-THREA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 scale=0.001 0.001 0.001
- link 94868A713_NO-THREADS_Female-Threaded-Hex-Standoff-3: geometry collision mesh filename=package://myrobot_sim_gazebo/urdf/meshes/94868A713_NO-THREA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 scale=0.001 0.001 0.001; visual mesh filename=package://myrobot_sim_gazebo/urdf/meshes/94868A713_NO-THREA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 scale=0.001 0.001 0.001
- link 94868A713_NO-THREADS_Female-Threaded-Hex-Standoff-4: geometry collision mesh filename=package://myrobot_sim_gazebo/urdf/meshes/94868A713_NO-THREA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 scale=0.001 0.001 0.001; visual mesh filename=package://myrobot_sim_gazebo/urdf/meshes/94868A713_NO-THREA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 scale=0.001 0.001 0.001
- link 94868A713_NO-THREADS_Female-Threaded-Hex-Standoff-5: geometry collision mesh filename=package://myrobot_sim_gazebo/urdf/meshes/94868A713_NO-THREA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 scale=0.001 0.001 0.001; visual mesh filename=package://myrobot_sim_gazebo/urdf/meshes/94868A713_NO-THREA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 scale=0.001 0.001 0.001
- link Base_08q-v1: geometry collision mesh filename=package://myrobot_sim_gazebo/urdf/meshes/Base_08q-v1.stl scale=0.001 0.001 0.001; visual mesh filename=package://myrobot_sim_gazebo/urdf/meshes/Base_08q-v1.stl scale=0.001 0.001 0.001
- link Battery---Battery-5.2-Ah-DC5521-Plug-v2: geometry collision mesh filename=package://myrobot_sim_gazebo/urdf/meshes/Battery---Battery-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 scale=0.001 0.001 0.001; visual mesh filename=package://myrobot_sim_gazebo/urdf/meshes/Battery---Battery-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 scale=0.001 0.001 0.001
- link Bottom-V2-v3: geometry collision mesh filename=package://myrobot_sim_gazebo/urdf/meshes/Bottom-V2-v3.stl scale=0.001 0.001 0.001; visual mesh filename=package://myrobot_sim_gazebo/urdf/meshes/Bottom-V2-v3.stl scale=0.001 0.001 0.001
- link Camera-Model-v3: geometry collision mesh filename=package://myrobot_sim_gazebo/urdf/meshes/Camera-Model-v3.stl scale=0.001 0.001 0.001; visual mesh filename=package://myrobot_sim_gazebo/urdf/meshes/Camera-Model-v3.stl scale=0.001 0.001 0.001
- link Camera-Model-v3-1: geometry collision mesh filename=package://myrobot_sim_gazebo/urdf/meshes/Camera-Model-v3-1.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 scale=0.001 0.001 0.001; visual mesh filename=package://myrobot_sim_gazebo/urdf/meshes/Camera-Model-v3-1.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 scale=0.001 0.001 0.001
- link Camera-Mount-v8: geometry collision mesh filename=package://myrobot_sim_gazebo/urdf/meshes/Camera-Mount-v8.stl scale=0.001 0.001 0.001; visual mesh filename=package://myrobot_sim_gazebo/urdf/meshes/Camera-Mount-v8.stl scale=0.001 0.001 0.001
- link Moving_Jaw_08d-v1: geometry collision mesh filename=package://myrobot_sim_gazebo/urdf/meshes/Moving_Jaw_08d-v1.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 scale=0.001 0.001 0.001; visual mesh filename=package://myrobot_sim_gazebo/urdf/meshes/Moving_Jaw_08d-v1.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 scale=0.001 0.001 0.001
- link Passive_Horn_01-v1: geometry collision mesh filename=package://myrobot_sim_gazebo/urdf/meshes/Passive_Horn_01-v1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 scale=0.001 0.001 0.001; visual mesh filename=package://myrobot_sim_gazebo/urdf/meshes/Passive_Horn_01-v1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 scale=0.001 0.001 0.001
- link Rotation_Pitch_08i-v1: geometry collision mesh filename=package://myrobot_sim_gazebo/urdf/meshes/Rotation_Pitch_08i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 scale=0.001 0.001 0.001; visual mesh filename=package://myrobot_sim_gazebo/urdf/meshes/Rotation_Pitch_08i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 scale=0.001 0.001 0.001
- link SO_ARM100_08k_116_Square-v1: geometry collision mesh filename=package://myrobot_sim_gazebo/urdf/meshes/SO_ARM100_08k_116_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 scale=0.001 0.001 0.001; visual mesh filename=package://myrobot_sim_gazebo/urdf/meshes/SO_ARM100_08k_116_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 scale=0.001 0.001 0.001
- link SO_ARM100_08k_Asym_Mirror_Clip-v1: geometry collision mesh filename=package://myrobot_sim_gazebo/urdf/meshes/SO_ARM100_08k_Asym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 scale=0.001 0.001 0.001; visual mesh filename=package://myrobot_sim_gazebo/urdf/meshes/SO_ARM100_08k_Asym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 scale=0.001 0.001 0.001
- link SO_ARM100_08k_Mirror-v1: geometry collision mesh filename=package://myrobot_sim_gazebo/urdf/meshes/SO_ARM100_08k_Mirr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 scale=0.001 0.001 0.001; visual mesh filename=package://myrobot_sim_gazebo/urdf/meshes/SO_ARM100_08k_Mirr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 scale=0.001 0.001 0.001
- link ST3215_Servo_Motor-v1: geometry collision mesh filename=package://myrobot_sim_gazebo/urdf/meshes/ST3215_Servo_Motor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 scale=0.001 0.001 0.001; visual mesh filename=package://myrobot_sim_gazebo/urdf/meshes/ST3215_Servo_Motor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 scale=0.001 0.001 0.001
- link ST3215_Servo_Motor-v1-1: geometry collision mesh filename=package://myrobot_sim_gazebo/urdf/meshes/ST3215_Servo_Motor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 scale=0.001 0.001 0.001; visual mesh filename=package://myrobot_sim_gazebo/urdf/meshes/ST3215_Servo_Motor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 scale=0.001 0.001 0.001
- link ST3215_Servo_Motor-v1-2: geometry collision mesh filename=package://myrobot_sim_gazebo/urdf/meshes/ST3215_Servo_Motor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 scale=0.001 0.001 0.001; visual mesh filename=package://myrobot_sim_gazebo/urdf/meshes/ST3215_Servo_Motor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 scale=0.001 0.001 0.001
- link STS3215_03a-v1: geometry collision mesh filename=package://myrobot_sim_gazebo/urdf/meshes/STS3215_03a-v1.stl scale=0.001 0.001 0.001; visual mesh filename=package://myrobot_sim_gazebo/urdf/meshes/STS3215_03a-v1.stl scale=0.001 0.001 0.001
- link STS3215_03a-v1-1: geometry collision mesh filename=package://myrobot_sim_gazebo/urdf/meshes/STS3215_03a-v1-1.s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 scale=0.001 0.001 0.001; visual mesh filename=package://myrobot_sim_gazebo/urdf/meshes/STS3215_03a-v1-1.s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 scale=0.001 0.001 0.001
- link STS3215_03a-v1-2: geometry collision mesh filename=package://myrobot_sim_gazebo/urdf/meshes/STS3215_03a-v1-2.s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 scale=0.001 0.001 0.001; visual mesh filename=package://myrobot_sim_gazebo/urdf/meshes/STS3215_03a-v1-2.s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 scale=0.001 0.001 0.001
- link STS3215_03a-v1-3: geometry collision mesh filename=package://myrobot_sim_gazebo/urdf/meshes/STS3215_03a-v1-3.s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 scale=0.001 0.001 0.001; visual mesh filename=package://myrobot_sim_gazebo/urdf/meshes/STS3215_03a-v1-3.s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 scale=0.001 0.001 0.001
- link STS3215_03a-v1-4: geometry collision mesh filename=package://myrobot_sim_gazebo/urdf/meshes/STS3215_03a-v1-4.s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 scale=0.001 0.001 0.001; visual mesh filename=package://myrobot_sim_gazebo/urdf/meshes/STS3215_03a-v1-4.s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 scale=0.001 0.001 0.001
- link STS3215_03a_Wrist_Roll-v1: geometry collision mesh filename=package://myrobot_sim_gazebo/urdf/meshes/STS3215_03a_Wrist_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 scale=0.001 0.001 0.001; visual mesh filename=package://myrobot_sim_gazebo/urdf/meshes/STS3215_03a_Wrist_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 scale=0.001 0.001 0.001
- link Top-V2-v2: geometry collision mesh filename=package://myrobot_sim_gazebo/urdf/meshes/Top-V2-v2.stl scale=0.001 0.001 0.001; visual mesh filename=package://myrobot_sim_gazebo/urdf/meshes/Top-V2-v2.stl scale=0.001 0.001 0.001
- link WaveShare_Mounting_Plate_01d-v1: geometry collision mesh filename=package://myrobot_sim_gazebo/urdf/meshes/WaveShare_Mounting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 scale=0.001 0.001 0.001; visual mesh filename=package://myrobot_sim_gazebo/urdf/meshes/WaveShare_Mounting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 scale=0.001 0.001 0.001
- link Wrist-Camera-Mount-v11: geometry collision mesh filename=package://myrobot_sim_gazebo/urdf/meshes/Wrist-Camera-Mount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 scale=0.001 0.001 0.001; visual mesh filename=package://myrobot_sim_gazebo/urdf/meshes/Wrist-Camera-Mount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 scale=0.001 0.001 0.001
- link Wrist_Roll_08c-v1: geometry collision mesh filename=package://myrobot_sim_gazebo/urdf/meshes/Wrist_Roll_08c-v1.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 scale=0.001 0.001 0.001; visual mesh filename=package://myrobot_sim_gazebo/urdf/meshes/Wrist_Roll_08c-v1.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 scale=0.001 0.001 0.001
- link Wrist_Roll_Pitch_08i-v1: geometry collision mesh filename=package://myrobot_sim_gazebo/urdf/meshes/Wrist_Roll_Pitch_0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 scale=0.001 0.001 0.001; visual mesh filename=package://myrobot_sim_gazebo/urdf/meshes/Wrist_Roll_Pitch_0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 scale=0.001 0.001 0.001
- link base_plate_layer1-v5: geometry collision mesh filename=package://myrobot_sim_gazebo/urdf/meshes/base_plate_layer1-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 scale=0.001 0.001 0.001; visual mesh filename=package://myrobot_sim_gazebo/urdf/meshes/base_plate_layer1-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 scale=0.001 0.001 0.001
- link base_plate_layer2-v3: geometry collision mesh filename=package://myrobot_sim_gazebo/urdf/meshes/base_plate_layer2-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 scale=0.001 0.001 0.001; visual mesh filename=package://myrobot_sim_gazebo/urdf/meshes/base_plate_layer2-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 scale=0.001 0.001 0.001
- link drive_motor_mount-v11: geometry collision mesh filename=package://myrobot_sim_gazebo/urdf/meshes/drive_motor_mount-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 scale=0.001 0.001 0.001; visual mesh filename=package://myrobot_sim_gazebo/urdf/meshes/drive_motor_mount-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 scale=0.001 0.001 0.001
- link drive_motor_mount-v11-1: geometry collision mesh filename=package://myrobot_sim_gazebo/urdf/meshes/drive_motor_mount-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 scale=0.001 0.001 0.001; visual mesh filename=package://myrobot_sim_gazebo/urdf/meshes/drive_motor_mount-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 scale=0.001 0.001 0.001
- link drive_motor_mount-v11-2: geometry collision mesh filename=package://myrobot_sim_gazebo/urdf/meshes/drive_motor_mount-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 scale=0.001 0.001 0.001; visual mesh filename=package://myrobot_sim_gazebo/urdf/meshes/drive_motor_mount-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 scale=0.001 0.001 0.001
- link lipo_battery_mount-v3: geometry collision mesh filename=package://myrobot_sim_gazebo/urdf/meshes/lipo_battery_mount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 scale=0.001 0.001 0.001; visual mesh filename=package://myrobot_sim_gazebo/urdf/meshes/lipo_battery_mount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 scale=0.001 0.001 0.001
- link omni_wheel_mount-v5: geometry collision mesh filename=package://myrobot_sim_gazebo/urdf/meshes/omni_wheel_mount-v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 scale=0.001 0.001 0.001; visual mesh filename=package://myrobot_sim_gazebo/urdf/meshes/omni_wheel_mount-v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 scale=0.001 0.001 0.001
- link omni_wheel_mount-v5-1: geometry collision mesh filename=package://myrobot_sim_gazebo/urdf/meshes/omni_wheel_mount-v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 scale=0.001 0.001 0.001; visual mesh filename=package://myrobot_sim_gazebo/urdf/meshes/omni_wheel_mount-v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 scale=0.001 0.001 0.001
- link omni_wheel_mount-v5-2: geometry collision mesh filename=package://myrobot_sim_gazebo/urdf/meshes/omni_wheel_mount-v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 scale=0.001 0.001 0.001; visual mesh filename=package://myrobot_sim_gazebo/urdf/meshes/omni_wheel_mount-v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 scale=0.001 0.001 0.001
- link servo_controller_mount-v3: geometry collision mesh filename=package://myrobot_sim_gazebo/urdf/meshes/servo_controller_m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 scale=0.001 0.001 0.001; visual mesh filename=package://myrobot_sim_gazebo/urdf/meshes/servo_controller_m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 scale=0.001 0.001 0.001

File: myrobot_sim_gazebo/urdf/turtlebot3_waffle.urdf (robot description, URDF)
Before this commit: robot turtlebot3_waffle, 13 links, 12 joints
Links:
- link base_link: geometry collision box size=0.266 0.266 0.094; visual mesh filename=package://myrobot_sim_gazebo/models/turtlebot3_common/meshe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 scale=0.001 0.001 0.001
- link base_scan: geometry collision cylinder length=0.0315 radius=0.055; visual mesh filename=package://myrobot_sim_gazebo/models/turtlebot3_common/meshe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 scale=0.001 0.001 0.001
- link camera_link: geometry collision box size=0.012 0.132 0.020; visual mesh filename=package://myrobot_sim_gazebo/models/turtlebot3_common/meshe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
- link wheel_left_link: geometry collision cylinder length=0.018 radius=0.033; visual mesh filename=package://myrobot_sim_gazebo/models/turtlebot3_common/meshe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 scale=0.001 0.001 0.001
- link wheel_right_link: geometry collision cylinder length=0.018 radius=0.033; visual mesh filename=package://myrobot_sim_gazebo/models/turtlebot3_common/meshe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 scale=0.001 0.001 0.001

File: myrobot_sim_gazebo/xacro/myrobot_diff_lidar_only.xacro (robot description, xacro)
@@ -1,4 +1,4 @@
 <?xml version="1.0"?>
-<robot name="lekiwi_diff_bot"
+<robot name="myrobot_diff_bot"
     xmlns:xacro="http://ros.org/wiki/xacro">
     <!-- PROPERTY LIST -->

File: myrobot_sim_gazebo/xacro/myrobot_diff_rgbd_only.xacro (robot description, xacro)
@@ -1,4 +1,4 @@
 <?xml version="1.0"?>
-<robot name="lekiwi_diff_bot"
+<robot name="myrobot_diff_bot"
     xmlns:xacro="http://ros.org/wiki/xacro">
     <!-- PROPERTY LIST -->

File: myrobot_sim_gazebo/xacro/myrobot_three_wheel.xacro (robot description, xacro)
@@ -18,5 +18,4 @@
         </inertial>
     </xacro:macro>
-    <!-- <xacro:include filename="$(find lekiwi_sim_gazebo)/xacro/lekiwi_wheel.xacro" /> -->
     <!-- PROPERTY LIST -->
     <xacro:property name="M_PI" value="3.1415926"/>
@@ -175,5 +174,5 @@
     <gazebo>
         <plugin name="gazebo_ros2_control" filename="libgazebo_ros2_control.so">
-            <parameters>$(find lekiwi_sim_gazebo)/config/my_robot_controllers.yaml</parameters>
+            <parameters>$(find myrobot_sim_gazebo)/config/my_robot_controllers.yaml</parameters>
         </plugin>
     </gazebo>

File: myrobot_sim_gazebo/xacro/myrobot_three_wheel_dev.xacro (robot description, xacro)
@@ -91,5 +91,5 @@
                 <origin xyz=" 0 0 0" rpy="0 0 0" />
                 <geometry>
-                    <mesh filename="file://$(find lekiwi_sim_gazebo)/meshes/mec_tiny_2.STL" scale="0.001 0.001 0.001"/>
+                    <mesh filename="file://$(find myrobot_sim_gazebo)/meshes/mec_tiny_2.STL" scale="0.001 0.001 0.001"/>
                 </geometry>
             </visual>
@@ -97,5 +97,5 @@
                 <origin xyz=" 0 0 0" rpy="0 0 0" />
                 <geometry>
-                    <mesh filename="file://$(find lekiwi_sim_gazebo)/meshes/mec_tiny_2.STL" scale="0.001 0.001 0.001"/>
+                    <mesh filename="file://$(find myrobot_sim_gazebo)/meshes/mec_tiny_2.STL" scale="0.001 0.001 0.001"/>
                     <!-- <cylinder radius="${tiny_wheel_radius}" length="${tiny_wheel_height}"/> -->
                 </geometry>
@@ -240,5 +240,5 @@
     <gazebo>
         <plugin name="gazebo_ros2_control" filename="libgazebo_ros2_control.so">
-            <parameters>$(find lekiwi_sim_gazebo)/config/my_robot_controllers.yaml</parameters>
+            <parameters>$(find myrobot_sim_gazebo)/config/my_robot_controllers.yaml</parameters>
         </plugin>
         <plugin name="joint_state_publisher" filename="libgazebo_ros_joint_state_publisher.so">
