Commit message: Opt sim

File: myrobot_sim_gazebo/xacro/myrobot_base.xacro (robot description, xacro)
@@ -1,4 +1,4 @@
 <?xml version="1.0"?>
-<robot name="jobot" xmlns:xacro="http://www.ros.org/wiki/xacro">
+<robot name="myrobot_base" xmlns:xacro="http://www.ros.org/wiki/xacro">
     <!-- PROPERTY LIST -->
     <xacro:property name="M_PI" value="3.1415926"/>

File: myrobot_sim_gazebo/xacro/sensor/camera_gazebo.xacro (robot description, xacro)
@@ -14,5 +14,5 @@
                 <origin xyz=" 0 0 0 " rpy="0 0 0" />
                 <geometry>
-                    <box size="0.04 0.055 0.04" />
+                    <box size="0.02 0.02 0.02" />
                 </geometry>
                 <material name="black"/>
@@ -21,5 +21,5 @@
                 <origin xyz="0.0 0.0 0.0" rpy="0 0 0" />
                 <geometry>
-                    <box size="0.04 0.055 0.04" />
+                    <box size="0.02 0.02 0.02" />
                 </geometry>
             </collision>
@@ -29,5 +29,5 @@
         </gazebo>
         <gazebo reference="${prefix}_link">
-            <sensor type="camera" name="camera_node">
+            <sensor type="${prefix}" name="camera_node">
                 <update_rate>30.0</update_rate>
                 <camera name="head">
@@ -51,6 +51,6 @@
 				    <ros>
 				        <!-- <namespace>stereo</namespace> -->
-				        <remapping>~/image_raw:=image_raw</remapping>
-				        <remapping>~/camera_info:=camera_info</remapping>
+				        <!-- <remapping>~/image_raw:=image_raw</remapping>
+				        <remapping>~/camera_info:=camera_info</remapping> -->
 				    </ros>
 				    <camera_name>${prefix}</camera_name>

File: myrobot_sim_gazebo/xacro/sensor/lidar_gazebo.xacro (robot description, xacro)
@@ -43,5 +43,5 @@
                     <range>
                       <min>0.10</min>
-                      <max>30.0</max>
+                      <max>15.0</max>
                       <resolution>0.01</resolution>
                     </range>
@@ -58,4 +58,5 @@
                     </ros>
                     <output_type>sensor_msgs/LaserScan</output_type>
+                    <frame_name>${prefix}_link</frame_name>
                 </plugin>
             </sensor>

File: myrobot_sim_gazebo/xacro/sensor/rgbd_gazebo.xacro (robot description, xacro)
@@ -14,19 +14,19 @@
         </link>
         <joint name="${prefix}_optical_joint" type="fixed">
-            <origin xyz="0 0 0" rpy="0 0 0"/>
+            <origin xyz="0 0 0" rpy="${-pi/2} 0 ${-pi/2}"/>
             <parent link="${prefix}_link"/>
-            <child link="${prefix}_rgb_optical_frame"/>
+            <child link="${prefix}_optical_frame"/>
         </joint>
-        <!-- <link name="${prefix}_rgb_optical_frame"/> -->
-        <link name="${prefix}_rgb_optical_frame">
+        <link name="${prefix}_optical_frame">
             <origin xyz="0 0 0" rpy="0 0 0"/>
         </link>
-        <gazebo reference="${prefix}_rgb_optical_frame">
+        <gazebo reference="${prefix}_link">
+        <!-- 这里的${prefix}决定话题名 /camera/depth/camera_info -->
             <sensor type="depth" name="${prefix}">
                 <always_on>true</always_on>
                 <visualize>true</visualize>
-                <update_rate>20.0</update_rate>
-                <camera name="intel_realsense_r200">
-                    <horizontal_fov>${60.0*M_PI/180.0}</horizontal_fov>
+                <update_rate>30.0</update_rate>
+                <camera name="${prefix}">
+                    <horizontal_fov>${60.0*pi/180.0}</horizontal_fov>
                     <image>
                         <format>R8G8B8</format>
@@ -36,5 +36,5 @@
                     <clip>
                         <near>0.02</near>
-                        <far>300</far>
+                        <far>8</far>
                     </clip>
                     <noise>
@@ -45,17 +45,20 @@
                 </camera>
                 <plugin name="${prefix}_controller" filename="libgazebo_ros_camera.so">
-		 		 	<ros>
-						<!-- <namespace>${prefix}</namespace> -->
-						<!-- <remapping>${prefix}/image_raw:=camera/image_raw</remapping>
-						<remapping>${prefix}/image_depth:=depth/image_raw</remapping>
-						<remapping>${prefix}/camera_info:=camera/camera_info</remapping>
-						<remapping>${prefix}/camera_info_depth:=depth/camera_info</remapping>
-						<remapping>${prefix}/points:=depth/points</remapping> -->
-					</ros>
-					<!-- <camera_name>${prefix}</camera_name>
-					<frame_name>${prefix}_rgb_optical_frame</frame_name>
-				    <hack_baseline>0.07</hack_baseline>
-				    <min_depth>0.001</min_depth>
-				    <max_depth>300.0</max_depth> -->
+		 		 	<baseline>0.2</baseline>
+                    <alwaysOn>true</alwaysOn>
+                    <updateRate>20.0</updateRate>
+                    <frame_name>${prefix}_optical_frame</frame_name>
+                    <!-- <pointCloudCutoff>0.5</pointCloudCutoff>
+                    <pointCloudCutoffMax>3.0</pointCloudCutoffMax>
+                    <distortionK1>0</distortionK1>
+                    <distortionK2>0</distortionK2>
+                    <distortionK3>0</distortionK3>
+                    <distortionT1>0</distortionT1>
+                    <distortionT2>0</distortionT2>
+                    <CxPrime>0</CxPrime>
+                    <Cx>0</Cx>
+                    <Cy>0</Cy>
+                    <focalLength>0</focalLength>
+                    <hackBaseline>0</hackBaseline> -->
                 </plugin>
             </sensor>
