Commit message: Add carto 3d

File: myrobot_sim_gazebo/xacro/myrobot_3d_lidar.xacro (robot description, xacro)
@@ -29,7 +29,7 @@
         max_range="30.0"
         update_rate="10"
-        visualize="true"/>
+        visualize="false"/>
     <joint name="imu_joint" type="fixed">
-        <origin xyz="0 0 ${base_height/2+0.01}" rpy="0 0 0" />
+        <origin xyz="0 0 0" rpy="0 0 0" />
         <parent link="base_link"/>
         <child link="imu_link"/>
