Commit message: Update

File: myrobot_sim_gazebo/xacro/myrobot_3d_lidar_no_odom.xacro (robot description, xacro)
@@ -17,15 +17,17 @@
         <child link="lidar3d_link"/>
     </joint>
+    <!-- MID-360 approximation for Gazebo's uniform gpu_ray scanner:
+         500 * 40 * 10 Hz = 200,000 points/s. -->
     <xacro:lidar_3d
         prefix="lidar3d"
         topic="points"
-        samples="720"
-        vertical_samples="16"
+        samples="500"
+        vertical_samples="40"
         min_angle="-3.14159"
         max_angle="3.14159"
-        min_vertical_angle="-0.261799"
-        max_vertical_angle="0.261799"
+        min_vertical_angle="-0.122173"
+        max_vertical_angle="0.907571"
         min_range="0.10"
-        max_range="30.0"
+        max_range="40.0"
         update_rate="10"
         visualize="true"/>

File: myrobot_sim_gazebo/xacro/myrobot_rgbd2_no_odom.xacro (robot description, xacro)
@@ -4,8 +4,9 @@
     <xacro:include filename="$(find myrobot_sim_gazebo)/xacro/sensor/rgbd_gazebo.xacro" />
     <xacro:include filename="$(find myrobot_sim_gazebo)/xacro/sensor/lidar_gazebo.xacro" />
+    <xacro:include filename="$(find myrobot_sim_gazebo)/xacro/sensor/imu_gazebo.xacro" />
     <xacro:property name="rgbd_offset_x" value="${base_radius+0.02}" />
     <xacro:property name="rgbd_offset_y" value="0" />
     <xacro:property name="rgbd_offset_z" value="0.02" />
-    <xacro:property name="lidar_offset_x" value="0" />
+    <xacro:property name="lidar_offset_x" value="0.07" />
     <xacro:property name="lidar_offset_y" value="0" />
     <xacro:property name="lidar_offset_z" value="${base_height/2+0.01}" />
@@ -27,3 +28,10 @@
     </joint>
     <xacro:lidar prefix="laser"/>
+    <!-- imu -->
+    <joint name="imu_joint" type="fixed">
+        <origin xyz="0 0 ${base_height/2+0.01}" rpy="0 0 0" />
+        <parent link="base_link"/>
+        <child link="imu_link"/>
+    </joint>
+    <xacro:imu_xacro prefix="imu"/>
 </robot>

File: myrobot_sim_gazebo/xacro/sensor/lidar_3d_gazebo.xacro (robot description, xacro)
@@ -4,14 +4,15 @@
         <link name="${prefix}_link">
             <inertial>
-                <mass value="0.25" />
+                <!-- Livox MID-360: 65 x 65 x 60 mm, 265 g. -->
+                <mass value="0.265" />
                 <origin xyz="0 0 0" />
-                <inertia ixx="0.02" ixy="0.0" ixz="0.0"
-                         iyy="0.02" iyz="0.0"
-                         izz="0.02" />
+                <inertia ixx="0.000172802" ixy="0.0" ixz="0.0"
+                         iyy="0.000172802" iyz="0.0"
+                         izz="0.000186604" />
             </inertial>
             <visual>
                 <origin xyz="0 0 0" rpy="0 0 0" />
                 <geometry>
-                    <cylinder length="0.05" radius="0.04"/>
+                    <box size="0.065 0.065 0.060"/>
                 </geometry>
                 <material name="black"/>
@@ -20,5 +21,5 @@
                 <origin xyz="0 0 0" rpy="0 0 0" />
                 <geometry>
-                    <cylinder length="0.05" radius="0.04"/>
+                    <box size="0.065 0.065 0.060"/>
                 </geometry>
             </collision>
